File: KICAD/Reforge_1.kicad_sch (KiCad schematic)
At the start: 90 parts, among them J1 USB_B_Micro, J2 Conn_01x19, J3 Conn_01x02, J4 Conn_01x24, J5 Conn_01x24, J8 Conn_01x19, Q1 SS8050, Q2 SS8050, SW1 SW_Push, SW2 SW_Push, U1 ESP32-WROOM-32E, U2 CP2102N-Axx-xQFN28, U3 ICE40UP5K-SG48ITR, U4 AP2112K-1.2, U5 AP2112K-3.3, U6 SN74LV4T125, U7 SN74LVC1G125DRL, U8 W25Q32JVSS, Y1 SG-210STF

Commit message: ADDED PCB DESIGN,UPDATED SCHEMATIC AND SOME MASTER & SLAVE SPI COMMUNICATION CODES THAT WE EXECUTED.
Parts:
- removed D3, D4, D5: D_TVS_Filled, Diode_SMD:D_SOD-323, symbol Device:D_TVS_Filled
- removed J1: USB_B_Micro, Connector_USB:USB_Micro-B_Molex_47346-0001, symbol Connector:USB_B_Micro
- removed J2, J8: Conn_01x19, Connector_PinHeader_2.54mm:PinHeader_1x19_P2.54mm_Horizontal, symbol Connector_Generic:Conn_01x19
- removed J4, J5: Conn_01x24, Connector_PinHeader_2.54mm:PinHeader_1x24_P2.54mm_Horizontal, symbol Connector_Generic:Conn_01x24
- removed TP6: TestPoint, TestPoint:TestPoint_Pad_D1.0mm, symbol Connector:TestPoint
- removed U1: ESP32-WROOM-32E, RF_Module:ESP32-WROOM-32E, symbol RF_Module:ESP32-WROOM-32E
- removed U5: AP2112K-3.3, Package_TO_SOT_SMD:SOT-23-5, symbol Regulator_Linear:AP2112K-3.3
- removed U6: SN74LV4T125, Package_SO:TSSOP-14_4.4x5mm_P0.65mm, symbol 74xx:SN74LV4T125
- removed U7: SN74LVC1G125DRL, Package_TO_SOT_SMD:Texas_R-PDSO-N5_DRL-5, symbol 74xGxx:SN74LVC1G125DRL
- added D3: SP0503BAHT, Package_TO_SOT_SMD:SOT-143, symbol Power_Protection:SP0503BAHT
- added J1: USB_C_Receptacle_USB2.0_16P, Connector_USB:USB_C_Receptacle_GCT_USB4105-xx-A_16P_TopMnt_Horizontal, symbol Connector:USB_C_Receptacle_USB2.0_16P
- added J10, J9: Conn_01x14_Pin, Connector_PinHeader_2.54mm:PinHeader_1x14_P2.54mm_Vertical, symbol Connector:Conn_01x14_Pin
- added J11, J12, J14, J15, J8: Conn_01x12_Pin, Connector_PinHeader_2.54mm:PinHeader_1x12_P2.54mm_Vertical, symbol Connector:Conn_01x12_Pin
- added R24, R25: 5.1K, Resistor_SMD:R_0805_2012Metric_Pad1.20x1.40mm_HandSolder, symbol Device:R
- added R26: 10K(5%), Resistor_SMD:R_0805_2012Metric_Pad1.20x1.40mm_HandSolder, symbol Device:R_Small_US
- added TP8: TestPoint, TestPoint:TestPoint_Pad_D1.0mm, symbol Connector:TestPoint
- added U11: SN74LVC2G125DCUR, SN74:SOP50P310X90-8N, symbol SN74LVC2G125DCUR:SN74LVC2G125DCUR
- added U5: ESP32-WROOM-32D, RF_Module:ESP32-WROOM-32D, symbol RF_Module:ESP32-WROOM-32D
- added U6: AMS1117-3.3, Package_TO_SOT_SMD:SOT-223-3_TabPin2, symbol Regulator_Linear:AMS1117-3.3
- C10, C11, C12, C14, C17, C18, C2, C20, C21, C24, C25, C26, C27, C28, C3, C9: footprint Capacitor_SMD:C_0402_1005Metric -> Capacitor_SMD:C_0805_2012Metric
- C13, C15, C16, C19, C22, C23, C6, C7, C8: footprint Capacitor_SMD:C_0603_1608Metric -> Capacitor_SMD:C_0805_2012Metric
- C4: value 22uF/10V(20%) -> 22uF
- C5: value 22uF/10V(20%) -> 10uF
- D6: value BAT760-7 -> SS14
- R1, R10, R11, R12, R14, R15, R18, R19, R2, R21, R22, R23, R3, R4, R5, R6, R7, R8, R9: footprint Resistor_SMD:R_0402_1005Metric -> Resistor_SMD:R_0805_2012Metric_Pad1.20x1.40mm_HandSolder
- R16, R17: value R -> 10K; footprint Resistor_SMD:R_0402_1005Metric -> Resistor_SMD:R_0805_2012Metric_Pad1.20x1.40mm_HandSolder
- SW1, SW2: footprint Button_Switch_SMD:SW_SPST_B3U-1000P -> Button_Switch_SMD:SW_Push_SPST_NO_Alps_SKRK
Connections:
- net +1V2 is gone; now on net +1.2V_CORE: R12.1
- net +1.2V_CORE: now also J11.5 (Pin_5), J14.7 (Pin_7)
- net +2V5: now also J15.1 (Pin_1)
- net CDONE: now also J11.7 (Pin_7)
- net CLK: now also J12.11 (Pin_11)
- net CLK_EXT: now also U11.3 (2Y)
- net CLK_FT: now also U11.2 (1A), U11.5 (2A)
- net CRESET_N: now also J11.8 (Pin_8)
- net CS: now also J10.10 (Pin_10), U5.29 (IO5)
- net EN: now also J9.3 (Pin_3), U5.3 (EN)
- net EXT_5V: now also J12.12 (Pin_12), U6.3 (VI); no longer C6.1, U4.1 (VIN)
- net FPGA_SI: now also J15.8 (Pin_8)
- net FPGA_SO: now also J15.11 (Pin_11)
- net FT_SCK: now also J15.10 (Pin_10)
- net FT_SSn: now also J15.9 (Pin_9)
- net GND: now also D3.1 (A), J1.A1 (GND), J1.A12 (GND), J1.B1 (GND), J1.B12 (GND), J1.SH (SHIELD), J10.1 (Pin_1), J10.7 (Pin_7), J12.1 (Pin_1), J9.1 (Pin_1), R24.2, R25.2, U11.1 (~{1OE}), U11.4 (GND), U11.7 (~{2OE}), U5.1 (GND), U5.15 (GND), U5.38 (GND), U5.39 (GND), U6.1 (GND)
- net IO0: now also J10.14 (Pin_14), R26.2, U5.25 (IO0)
- net IO12: now also J9.14 (Pin_14), U5.14 (IO12)
- net IO13: now also J12.2 (Pin_2), U5.16 (IO13)
- net IO14: now also J9.13 (Pin_13), U5.13 (IO14)
- net IO15: now also J12.9 (Pin_9), U5.23 (IO15)
- net IO16: now also J10.12 (Pin_12), U5.27 (IO16)
- net IO17: now also J10.11 (Pin_11), U5.28 (IO17)
- net IO2: now also J12.10 (Pin_10), U5.24 (IO2)
- net IO21: now also J10.6 (Pin_6), U5.33 (IO21)
- net IO22: now also J10.3 (Pin_3), U5.36 (IO22)
- net IO25: now also J9.10 (Pin_10), U5.10 (IO25)
- net IO26: now also J9.11 (Pin_11), U5.11 (IO26)
- net IO27: now also J9.12 (Pin_12), U5.12 (IO27)
- net IO32: now also J9.8 (Pin_8), U5.8 (IO32)
- net IO33: now also J9.9 (Pin_9), U5.9 (IO33)
- net IO34: now also J9.6 (Pin_6), U5.6 (IO34)
- net IO35: now also J9.7 (Pin_7), U5.7 (IO35)
- net IO4: now also J10.13 (Pin_13), U5.26 (IO4)
- net IOB_0A: now also J8.10 (Pin_10)
- net IOB_13B: now also J11.6 (Pin_6)
- net IOB_16A: now also J11.9 (Pin_9)
- net IOB_18A: now also J11.10 (Pin_10)
- net IOB_20A: now also J11.11 (Pin_11)
- net IOB_22A: now also J11.12 (Pin_12)
- net IOB_23B: now also J15.4 (Pin_4)
- net IOB_24A: now also J15.12 (Pin_12)
- net IOB_25B_G3: now also SJ27.2, J15.5 (Pin_5); no longer SJ27.1
- net IOB_29B: now also J15.6 (Pin_6)
- net IOB_2A: now also J8.11 (Pin_11)
- net IOB_31B: now also J15.7 (Pin_7)
- net IOB_3B_G6: now also J8.8 (Pin_8)
- net IOB_4A: now also J8.12 (Pin_12)
- net IOB_5B: now also J8.9 (Pin_9)
- net IOB_6A: now also J11.2 (Pin_2)
- net IOB_8A: now also J11.4 (Pin_4)
- net IOB_9B: now also J11.3 (Pin_3)
- net IOT_36B: now also J14.12 (Pin_12)
- net IOT_37A: now also J15.2 (Pin_2)
- net IOT_38B: now also J14.10 (Pin_10)
- net IOT_39A: now also J14.11 (Pin_11)
- net IOT_41A: now also J14.9 (Pin_9)
- net IOT_42B: now also J14.6 (Pin_6)
- net IOT_43A: now also J14.5 (Pin_5)
- net IOT_44B: now also J14.3 (Pin_3)
- net IOT_45A_G1: now also J8.1 (Pin_1)
- net IOT_46B_G0: now also J14.2 (Pin_2)
- net IOT_48B: now also J14.1 (Pin_1)
- net IOT_49A: now also J8.7 (Pin_7)
- net IOT_50B: now also J8.2 (Pin_2)
- net IOT_51A: now also J8.6 (Pin_6)
- net LED_B: now also J8.4 (Pin_4)
- net LED_G: now also J8.3 (Pin_3)
- net LED_R: now also J8.5 (Pin_5)
- net MISO: now also J10.8 (Pin_8), U5.31 (IO19)
- net MOSI: now also J10.2 (Pin_2), U5.37 (IO23)
- net RXD0: now also J10.5 (Pin_5), U5.34 (RXD0/IO3)
- net SCK: now also J10.9 (Pin_9), U5.30 (IO18)
- net SENSOR_VN: now also J9.5 (Pin_5), U5.5 (SENSOR_VN)
- net SENSOR_VP: now also J9.4 (Pin_4), U5.4 (SENSOR_VP)
- net TXD0: now also J10.4 (Pin_4), U5.35 (TXD0/IO1)
- net USB_DN: now also D3.3 (K), J1.A7 (D-), J1.B7 (D-)
- net USB_DP: now also D3.2 (K), J1.A6 (D+), J1.B6 (D+)
- net VBUS: now also D3.4 (K), J1.A4 (VBUS), J1.A9 (VBUS), J1.B4 (VBUS), J1.B9 (VBUS)
- net VCC_PLL: now also J14.8 (Pin_8)
- net VDD33: now also C6.1, U4.1 (VIN), J15.3 (Pin_3), J9.2 (Pin_2), R26.1, TP8.1, U11.8 (VCC), U5.2 (VDD), U6.2 (VO)
- net VCCIO_2: now reaches C16.1, C17.1, SJ20.2, SJ26.2, U3.1 (VCCIO_2)
- net VCCIO_2: now also J11.1 (Pin_1)
- net VCCIO_0: now reaches C12.1, C13.1, SJ19.2, SJ31.2, U3.33 (VCCIO_0)
- net VCCIO_0: now also J14.4 (Pin_4)
- new net: SJ27.1, U11.6 (1Y)
- new net: J1.A5 (CC1), R24.1
- new net: J1.B5 (CC2), R25.1
- new net SCK/CLK: J12.6 (Pin_6), U5.20 (SCK/CLK)
- new net SCS/CMD: J12.5 (Pin_5), U5.19 (SCS/CMD)
- new net SDI/SD1: J12.8 (Pin_8), U5.22 (SDI/SD1)
- new net SDO/SD0: J12.7 (Pin_7), U5.21 (SDO/SD0)
- new net SHD/SD2: J12.3 (Pin_3), U5.17 (SHD/SD2)
- new net SWP/SD3: J12.4 (Pin_4), U5.18 (SWP/SD3)
- no-connect marks 29 -> 16
Other:
- note added: "USB-C"
- note removed: "MICRO-USB"
- moved on the sheet: C10, C11, C24, C25, C26, C27, C28, C8, C9, D6, J3, Q1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

Commit message: Update schematic and PCB
Parts:
- removed C26, C27, C28: DNI, Capacitor_SMD:C_0805_2012Metric, symbol Device:C
- removed R7, R8: 0R(5%), Resistor_SMD:R_0805_2012Metric_Pad1.20x1.40mm_HandSolder, symbol Device:R_US
- removed TP1, TP2, TP8: TestPoint, TestPoint:TestPoint_Pad_D1.0mm, symbol Connector:TestPoint
- removed VBUS1: TestPoint, LED_SMD:LED_RGB_Wuerth-PLCC4_3.2x2.8mm_150141M173100, symbol Connector:TestPoint
- R20: footprint Resistor_SMD:R_0402_1005Metric -> Resistor_SMD:R_0805_2012Metric_Pad1.20x1.40mm_HandSolder
Connections:
- net TXD is gone; now on net RXD0: U2.26 (TXD)
- net TXD0 is gone; now on net RXD: J10.4 (Pin_4), U5.35 (TXD0/IO1)
- net IO0: now also Q2.3 (C); no longer Q2.2 (E)
- net ~{DTR}: now also Q2.2 (E); no longer Q2.3 (C)

Commit message: Added some more diodes and Placement done
Parts:
- added PWR_LED2, PWR_LED3: RED LED, LED_SMD:LED_0603_1608Metric, symbol Device:LED
- added R7: 330R, Resistor_SMD:R_0805_2012Metric_Pad1.20x1.40mm_HandSolder, symbol Device:R_US
- added R8: 1K, Resistor_SMD:R_0805_2012Metric_Pad1.20x1.40mm_HandSolder, symbol Device:R_US
- D6: footprint Diode_SMD:D_SOD-323 -> Diode_SMD:D_SMB
- R2: value 2K(5%) -> 330R
Connections:
- net FPGA_SI is gone; now on net MOSI: J15.8 (Pin_8), R22.2, R23.2, U3.17 (IOB_33b_SPI_SI)
- net FPGA_SO is gone; now on net MISO: J15.11 (Pin_11), R20.1, R21.2, U3.14 (IOB_32a_SPI_SO)
- net FT_SSn is gone; now on net CS: J15.9 (Pin_9), R16.2, U3.16 (IOB_35b_SPI_SS), U8.1 (~{CS})
- net CLK: now also J15.10 (Pin_10)
- net EXT_5V: now also R8.1; no longer R2.1
- net GND: now also PWR_LED2.1 (K), PWR_LED3.1 (K)
- net SCK: now also R17.2, U3.15 (IOB_34a_SPI_SCK), U8.6 (CLK)
- net VDD12: now also R7.1
- net VDD33: now also R2.1
- removed net FT_SCK: J15.10 (Pin_10), R17.2, U3.15 (IOB_34a_SPI_SCK), U8.6 (CLK)
- new net: PWR_LED3.2 (A), R8.2
- new net: PWR_LED2.2 (A), R7.2
Other:
- moved on the sheet: C4, C5, C6, C7, PWR_LED1, R2, U4, U6

Commit message: Did Routing and updates schematic
Parts:
- R8: value 1K -> 330R
Connections:
- net CLK: no longer J15.10 (Pin_10)
- net SCK: now also J15.10 (Pin_10)
- no-connect marks 16 -> 17
Changed lines of the file:
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@@
 	)
 	(junction
-		(at 541.02 43.18)
-		(diameter 0)
-		(color 0 0 0 0)
-	)
-	(junction
 		(at 204.47 93.98)
 		(diameter 0)
@@
 	)
 	(no_connect
+		(at 440.69 180.34)
+	)
+	(no_connect
 		(at 189.23 215.9)
 	)
@@
 	(wire
 		(pts
-			(xy 541.02 43.18) (xy 548.64 43.18)
+			(xy 537.21 43.18) (xy 548.64 43.18)
 		)
 		(stroke
@@
 	(wire
 		(pts
-			(xy 537.21 43.18) (xy 541.02 43.18)
-		)
-		(stroke
-			(width 0)
-			(type default)
-		)
-	)
-	(wire
-		(pts
 			(xy 179.07 243.84) (xy 189.23 243.84)
 		)
@@
 		)
 	)
-	(label "CLK"
+	(label "SCK"
 		(at 527.05 193.04 0)
 		(effects
@@
 		(lib_id "Device:R_US")
 		(at 212.09 60.96 0)
+		(mirror y)
 		(unit 1)
 		(body_style 1)
@@
 		(dnp no)
 		(property "Reference" "R2"
-			(at 213.614 57.404 0)
+			(at 210.566 57.404 0)
 			(show_name no)
 			(do_not_autoplace no)
@@
 		)
 		(property "Value" "330R"
-			(at 213.36 59.182 0)
+			(at 210.82 59.182 0)
 			(show_name no)
 			(do_not_autoplace no)
@@
 		)
 		(property "Footprint" "Resistor_SMD:R_0805_2012Metric_Pad1.20x1.40mm_HandSolder"
-			(at 213.106 61.214 90)
+			(at 211.074 61.214 90)
 			(hide yes)
 			(show_name no)
@@
 		(in_pos_files yes)
 		(dnp no)
-		(fields_autoplaced yes)
 		(property "Reference" "U8"
 			(at 374.65 251.4599 0)
@@
 		(in_pos_files yes)
 		(dnp no)
-		(fields_autoplaced yes)
 		(property "Reference" "D1"
 			(at 554.99 63.5 0)
@@
 					(size 1.27 1.27)
 				)
-				(justify left)
+				(justify right)
 			)
 		)
-		(property "Value" "1K"
+		(property "Value" "330R"
 			(at 102.87 191.262 0)
 			(show_name no)
@@
 					(unit 1)
 				)
-			)
-		)
-	)
-	(symbol
-		(lib_id "power:PWR_FLAG")
-		(at 541.02 43.18 180)
-		(unit 1)
-		(body_style 1)
-		(exclude_from_sim no)
-		(in_bom yes)
-		(on_board yes)
-		(in_pos_files yes)
-		(dnp no)
-		(property "Reference" "#FLG05"
-			(at 541.02 45.085 0)
-			(hide yes)
-			(show_name no)
-			(do_not_autoplace no)
-			(effects
-				(font
-					(size 1.27 1.27)
-				)
-			)
-		)
-		(property "Value" "PWR_FLAG"
-			(at 541.274 46.736 0)
-			(show_name no)
-			(do_not_autoplace no)
-			(effects
-				(font
-					(size 1.27 1.27)
-				)
-			)
-		)
-		(property "Footprint" ""
-			(at 541.02 43.18 0)
-			(hide yes)
-			(show_name no)
-			(do_not_autoplace no)
-			(effects
-				(font
-					(size 1.27 1.27)
-				)
-			)
-		)
-		(property "Datasheet" ""
-			(at 541.02 43.18 0)
-			(hide yes)
-			(show_name no)
-			(do_not_autoplace no)
-			(effects
-				(font
-					(size 1.27 1.27)
-				)
-			)
-		)
-		(property "Description" "Special symbol for telling ERC where power comes from"
-			(at 541.02 43.18 0)
-			(hide yes)
-			(show_name no)
-			(do_not_autoplace no)
-			(effects
-				(font
-					(size 1.27 1.27)
-				)
-			)
-		)
-		(pin "1"
-		)
-		(instances
-			(project "Reforge_1"
-				(path "/ba70c426-5169-436b-9f8e-122ac1661c00"
-					(reference "#FLG05")
-					(unit 1)
-				)
