File: KICAD/Reforge_1.kicad_sch (KiCad schematic)
At the start: 88 parts, among them J1 USB_C_Receptacle_USB2.0_16P, J10 Conn_01x14_Pin, J11 Conn_01x12_Pin, J12 Conn_01x12_Pin, J14 Conn_01x12_Pin, J15 Conn_01x12_Pin, J3 Conn_01x02, J8 Conn_01x12_Pin, J9 Conn_01x14_Pin, Q1 SS8050, Q2 SS8050, SW1 SW_Push, SW2 SW_Push, U11 SN74LVC2G125DCUR, U2 CP2102N-Axx-xQFN28, U3 ICE40UP5K-SG48ITR, U4 AP2112K-1.2, U5 ESP32-WROOM-32D, U6 AMS1117-3.3, U8 W25Q32JVSS, Y1 SG-210STF

Commit message: Updated Schematic, Added mounting hole and some updates in PCB
Parts:
- removed C5: 10uF, Capacitor_SMD:C_0805_2012Metric, symbol Device:C_Small
- added C26: 22uF, Capacitor_SMD:C_0805_2012Metric, symbol Device:C_Small
- added C27, C28: 0.1uF, Capacitor_SMD:C_0805_2012Metric, symbol Device:C_Small
- added H1: MountingHole, MountingHole:MountingHole_2.1mm, symbol Mechanical:MountingHole
- C4: value 22uF -> 10uF
- R10, R9: value 10R(5%) -> 10k(5%)
Connections:
- net EN: no longer U4.3 (EN)
- net EXT_5V: now also C28.2
- net GND: now also C26.2, C27.1, C28.1
- net VDD33: now also U4.3 (EN), C26.1, C27.2
Other:
- moved on the sheet: PWR_LED1, R2

Commit message: Updated PCB
Parts:
- C20: value 0.1uF -> 4.7uF
- SJ27: value OPEN -> SHORT
Changed lines of the file:
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@@
 			)
 		)
-		(property "Value" "OPEN"
-			(at 432.054 176.276 90)
+		(property "Value" "SHORT"
+			(at 432.816 176.276 90)
 			(show_name no)
 			(do_not_autoplace no)
@@
 			)
 		)
-		(property "Value" "0.1uF"
+		(property "Value" "4.7uF"
 			(at 508 74.93 0)
 			(show_name no)

Commit message: Updated PCB
Connections:
- net CLK renamed CP_CLK
Changed lines of the file:
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@@
 		)
 	)
-	(label "CLK"
+	(label "CP_CLK"
 		(at 321.31 252.73 180)
 		(effects
@@
 		)
 	)
-	(label "CLK"
+	(label "CP_CLK"
 		(at 189.23 226.06 180)
 		(effects
