File: KICAD/Reforge_1.kicad_pcb (KiCad board)
At the start: 2 copper layers, 61 x 77.8 mm, 95 parts, among them J1 USB_C_Receptacle_USB2.0_16P, J10 Conn_01x14_Pin, J11 Conn_01x12_Pin, J12 Conn_01x12_Pin, J14 Conn_01x12_Pin, J15 Conn_01x12_Pin, J3 Conn_01x02, J8 Conn_01x12_Pin, J9 Conn_01x14_Pin, Q1 SS8050, Q2 SS8050, SW1 SW_Push, SW2 SW_Push, U11 SN74LVC2G125DCUR, U2 CP2102N-Axx-xQFN28, U3 ICE40UP5K-SG48ITR, U4 AP2112K-1.2, U5 ESP32-WROOM-32D, U6 AMS1117-3.3, U8 W25Q32JVSS, Y1 SG-210STF

Commit message: Updated PCB
Parts:
- added G***: LOGO, LOGO, B.Cu at (151.4, 116.0)
- C20: value 0.1uF -> 4.7uF
- SJ27: value OPEN -> SHORT
- moved G*** 19.2 mm to (138.1, 95.8)
- moved C21 1.25 mm to (143.5, 94.9)
Routing:
- net /VDD33: track 316.5 -> 321.5 mm
- net /IOB_31B: track 47.3 -> 45.1 mm
- net /IO35: track 18.5 -> 20.3 mm
- net /IOB_23B: track 31.8 -> 33.6 mm
- net /IO34: track 16.8 -> 18.5 mm
- net /IO32: track 19.6 -> 21.3 mm
- net /IOB_29B: track 30.8 -> 32.4 mm
- net /SWP/SD3: track 12.4 -> 10.9 mm
- net /IOT_37A: track 30.2 -> 31.6 mm
- net /SCK: track 117.1 -> 118.5 mm
- net /IO33: track 20.8 -> 22.0 mm
- net /IOB_25B_G3: track 33.9 -> 35.1 mm
- net /SENSOR_VN: track 15.8 -> 16.9 mm
- net /SCS/CMD: track 11.4 -> 10.4 mm
- net /SHD/SD2: track 12.9 -> 12.0 mm
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Other:
- board text added: "CP_CLK"
- board text added: "TXD0"
- board text removed: "CLK"
- board text removed: "RXD"

Commit message: Updated PCB
Parts:
- moved SJ31 0.15 mm to (127.8, 97.1), turned to 0 degrees
Connections:
- net /CLK renamed /CP_CLK
Routing:
- net /VDD33: track 321.5 -> 311.5 mm, vias 27 -> 25
- net /EXT_5V: track 81.2 -> 75.9 mm
- net Net-(U8-~{HOLD}/~{RESET}/IO_{3}): track 13.5 -> 10.9 mm
- net /IOB_29B: track 32.4 -> 29.9 mm
- net /+1.2V_CORE: track 126.0 -> 124.3 mm
- net /IOT_51A: track 23.2 -> 21.9 mm
- net /IOB_23B: track 33.6 -> 32.3 mm
- net /FLASH_MISO: track 17.3 -> 18.5 mm
- net /IOB_9B: track 17.6 -> 16.8 mm
- net /IOT_45A_G1: track 18.8 -> 18.0 mm
- net /VCCIO_0: track 21.1 -> 20.4 mm
- net /IOT_48B: track 16.8 -> 16.1 mm
- net /IOT_46B_G0: track 16.1 -> 15.4 mm
- net /IOB_18A: track 35.3 -> 34.7 mm
- net /IOB_6A: track 19.2 -> 18.6 mm
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Other:
- board text added: "2026"
- board text added: "EKLAVYA"
